File: RFInput.brd (EAGLE design)
At the start: 100 x 80 mm, 10 parts, among them J1 BNCPTH

Commit message: commit
Parts:
- removed 5V, GND, OUT: (no value), wirepad:2,54/1,1
- added C4, C5, C6, C8: 0.001uF, SparkFun-Capacitors:1206
- added C7: 0.1uF, SparkFun-Capacitors:1206
- added J2: BNCPTH, SparkFun-Connectors:BNC
- added J3: (no value), SparkFun-Connectors:1X04
- added L2: 100uH, inductor-neosid:BS75
- added R2: 52.3, SparkFun-Resistors:0805
- added U$2: AD8307, SparkFun-IC-Amplifiers:SO08
- moved C3 1.27 mm to (43.2, 74.9)
- moved L1 1.27 mm to (43.2, 68.6)
- moved J1 1.27 mm to (12.7, 69.8)
Connections:
- removed net N$4: 5V.1, L1.2
- removed net N$5: OUT.1, U$1.4
- new net 5V: J3.4, L1.2, L2.2
- new net N$6: C5.1, J2.S, R2.2
- new net N$7: C5.2, U$2.8
- new net N$8: C6.2, U$2.1
- new net N$9: C7.2, L2.1, U$2.6, U$2.7
- new net OUT1: C4.2, J3.2, U$1.4
- new net OUT2: C8.2, J3.1, U$2.4
- net GND: now also C4.1, C6.1, C7.1, C8.1, J2.GND, J3.3, R2.1, U$2.2; no longer GND.1
Routing:
- net GND: track 48.6 -> 156.9 mm
- net OUT2: track 0.00 -> 39.5 mm
- net 5V: track 0.00 -> 34.2 mm
- net OUT1: track 0.00 -> 33.2 mm
- net N$9: track 0.00 -> 23.1 mm
- net N$5: track 17.2 -> 0.00 mm
- net N$6: track 0.00 -> 14.0 mm
- net N$4: track 8.93 -> 0.00 mm
- net N$8: track 0.00 -> 6.22 mm
- net N$7: track 0.00 -> 6.22 mm
- net N$12: track 12.7 -> 14.0 mm
