File: RFInput.sch (EAGLE design)
At the start: 10 parts, among them J1 BNCPTH

Commit message: commit
Parts:
- removed 5V, GND, OUT: (no value), wirepad:2,54/1,1
- added C4, C5, C6, C8: 0.001uF, SparkFun-Capacitors:1.0UF-1206-50V-10%
- added C7: 0.1uF, SparkFun-Capacitors:1.0UF-1206-50V-10%
- added J2: BNCPTH, SparkFun-Connectors:BNCPTH
- added J3: (no value), SparkFun-Connectors:CONN_04
- added L2: 100uH, inductor-neosid:BS75
- added R2: 52.3, SparkFun-Resistors:0.75OHM-0805-1/4W-1%
- added U$2: AD8307, SparkFun-IC-Amplifiers:AD8307
Connections:
- removed net N$4: 5V.P, L1.2
- removed net N$5: OUT.P, U$1.OUT
- new net 5V: J3.4, L1.2, L2.2
- new net N$6: C5.1, J2.OUT, R2.2
- new net N$7: C5.2, U$2.IN+
- new net N$8: C6.2, U$2.IN-
- new net N$9: C7.2, L2.1, U$2.ENB, U$2.VPS
- new net OUT1: C4.2, J3.2, U$1.OUT
- new net OUT2: C8.2, J3.1, U$2.OUT
- net GND: now also C4.1, C6.1, C7.1, C8.1, J2.GND, J3.3, R2.1, U$2.COM; no longer GND.P
Changed lines of the file:
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@@
 <part name="GND3" library="SparkFun-PowerSymbols" deviceset="GND" device=""/>
 <part name="L1" library="inductor-neosid" library_urn="urn:adsk.eagle:library:241" deviceset="BS" device="75" package3d_urn="urn:adsk.eagle:package:14660/1" value="100uH"/>
-<part name="5V" library="wirepad" library_urn="urn:adsk.eagle:library:412" deviceset="2,54/1,1" device="" package3d_urn="urn:adsk.eagle:package:30836/1"/>
-<part name="GND" library="wirepad" library_urn="urn:adsk.eagle:library:412" deviceset="2,54/1,1" device="" package3d_urn="urn:adsk.eagle:package:30836/1"/>
-<part name="OUT" library="wirepad" library_urn="urn:adsk.eagle:library:412" deviceset="2,54/1,1" device="" package3d_urn="urn:adsk.eagle:package:30836/1"/>
+<part name="C4" library="SparkFun-Capacitors" deviceset="1.0UF" device="-1206-50V-10%" value="0.001uF"/>
+<part name="GND4" library="SparkFun-PowerSymbols" deviceset="GND" device=""/>
+<part name="J2" library="SparkFun-Connectors" deviceset="BNC" device="PTH"/>
+<part name="GND5" library="SparkFun-PowerSymbols" deviceset="GND" device=""/>
+<part name="R2" library="SparkFun-Resistors" deviceset="0.75OHM" device="-0805-1/4W-1%" value="52.3"/>
+<part name="GND7" library="SparkFun-PowerSymbols" deviceset="GND" device=""/>
+<part name="C5" library="SparkFun-Capacitors" deviceset="1.0UF" device="-1206-50V-10%" value="0.001uF"/>
+<part name="C6" library="SparkFun-Capacitors" deviceset="1.0UF" device="-1206-50V-10%" value="0.001uF"/>
+<part name="U$2" library="SparkFun-IC-Amplifiers" deviceset="AD8307" device=""/>
+<part name="GND8" library="SparkFun-PowerSymbols" deviceset="GND" device=""/>
+<part name="C7" library="SparkFun-Capacitors" deviceset="1.0UF" device="-1206-50V-10%" value="0.1uF"/>
+<part name="GND9" library="SparkFun-PowerSymbols" deviceset="GND" device=""/>
+<part name="L2" library="inductor-neosid" library_urn="urn:adsk.eagle:library:241" deviceset="BS" device="75" package3d_urn="urn:adsk.eagle:package:14660/1" value="100uH"/>
+<part name="C8" library="SparkFun-Capacitors" deviceset="1.0UF" device="-1206-50V-10%" value="0.001uF"/>
+<part name="GND11" library="SparkFun-PowerSymbols" deviceset="GND" device=""/>
+<part name="J3" library="SparkFun-Connectors" deviceset="CONN_04" device=""/>
 </parts>
 <sheets>
@@
 <instance part="GND3" gate="1" x="58.42" y="71.12"/>
 <instance part="L1" gate="G$1" x="53.34" y="81.28" rot="R180"/>
-<instance part="5V" gate="1" x="27.94" y="81.28"/>
-<instance part="GND" gate="1" x="66.04" y="30.48" rot="R180"/>
-<instance part="OUT" gate="1" x="91.44" y="35.56" rot="R180"/>
+<instance part="C4" gate="G$1" x="81.28" y="33.02" rot="R180"/>
+<instance part="GND4" gate="1" x="81.28" y="25.4"/>
+<instance part="J2" gate="G$1" x="101.6" y="55.88"/>
+<instance part="GND5" gate="1" x="101.6" y="48.26"/>
+<instance part="R2" gate="G$1" x="119.38" y="50.8" rot="R90"/>
+<instance part="GND7" gate="1" x="119.38" y="43.18"/>
+<instance part="C5" gate="G$1" x="124.46" y="55.88" rot="R90"/>
+<instance part="C6" gate="G$1" x="124.46" y="45.72" rot="R90"/>
+<instance part="U$2" gate="G$1" x="152.4" y="53.34" rot="R90"/>
+<instance part="GND8" gate="1" x="152.4" y="27.94"/>
+<instance part="C7" gate="G$1" x="147.32" y="78.74" rot="R180"/>
+<instance part="GND9" gate="1" x="147.32" y="71.12"/>
+<instance part="L2" gate="G$1" x="142.24" y="81.28" rot="R180"/>
+<instance part="C8" gate="G$1" x="170.18" y="33.02" rot="R180"/>
+<instance part="GND11" gate="1" x="170.18" y="25.4"/>
+<instance part="J3" gate="G$1" x="93.98" y="88.9"/>
 </instances>
 <busses>
@@
 <pinref part="GND2" gate="1" pin="GND"/>
 <wire x1="63.5" y1="43.18" x2="63.5" y2="30.48" width="0.1524" layer="91"/>
-<pinref part="GND" gate="1" pin="P"/>
-<junction x="63.5" y="30.48"/>
 </segment>
 <segment>
 <pinref part="GND3" gate="1" pin="GND"/>
 <pinref part="C3" gate="G$1" pin="1"/>
+</segment>
+<segment>
+<pinref part="GND4" gate="1" pin="GND"/>
+<pinref part="C4" gate="G$1" pin="1"/>
+</segment>
+<segment>
+<pinref part="GND5" gate="1" pin="GND"/>
+<pinref part="J2" gate="G$1" pin="GND"/>
+</segment>
+<segment>
+<pinref part="GND7" gate="1" pin="GND"/>
+<pinref part="R2" gate="G$1" pin="1"/>
+<pinref part="C6" gate="G$1" pin="1"/>
+<junction x="119.38" y="45.72"/>
+</segment>
+<segment>
+<pinref part="U$2" gate="G$1" pin="COM"/>
+<pinref part="GND8" gate="1" pin="GND"/>
+<wire x1="152.4" y1="43.18" x2="152.4" y2="30.48" width="0.1524" layer="91"/>
+</segment>
+<segment>
+<pinref part="GND9" gate="1" pin="GND"/>
+<pinref part="C7" gate="G$1" pin="1"/>
+</segment>
+<segment>
+<pinref part="GND11" gate="1" pin="GND"/>
+<pinref part="C8" gate="G$1" pin="1"/>
+</segment>
+<segment>
+<pinref part="J3" gate="G$1" pin="3"/>
+<wire x1="99.06" y1="91.44" x2="104.14" y2="91.44" width="0.1524" layer="91"/>
+<label x="106.68" y="91.44" size="1.778" layer="95"/>
 </segment>
 </net>
@@
 </segment>
 </net>
-<net name="N$4" class="0">
-<segment>
-<pinref part="L1" gate="G$1" pin="2"/>
-<wire x1="48.26" y1="81.28" x2="30.48" y2="81.28" width="0.1524" layer="91"/>
-<pinref part="5V" gate="1" pin="P"/>
-</segment>
-</net>
-<net name="N$5" class="0">
+<net name="OUT1" class="0">
 <segment>
 <pinref part="U$1" gate="G$1" pin="OUT"/>
 <wire x1="68.58" y1="43.18" x2="68.58" y2="35.56" width="0.1524" layer="91"/>
-<wire x1="68.58" y1="35.56" x2="88.9" y2="35.56" width="0.1524" layer="91"/>
-<pinref part="OUT" gate="1" pin="P"/>
-</segment>
-</net>
+<wire x1="68.58" y1="35.56" x2="81.28" y2="35.56" width="0.1524" layer="91"/>
+<pinref part="C4" gate="G$1" pin="2"/>
+<wire x1="81.28" y1="35.56" x2="88.9" y2="35.56" width="0.1524" layer="91"/>
+<junction x="81.28" y="35.56"/>
+<label x="88.9" y="38.1" size="1.778" layer="95"/>
+</segment>
+<segment>
+<pinref part="J3" gate="G$1" pin="2"/>
+<wire x1="99.06" y1="88.9" x2="104.14" y2="88.9" width="0.1524" layer="91"/>
+<label x="106.68" y="88.9" size="1.778" layer="95"/>
+</segment>
+</net>
+<net name="N$6" class="0">
+<segment>
+<pinref part="J2" gate="G$1" pin="OUT"/>
+<wire x1="119.38" y1="55.88" x2="106.68" y2="55.88" width="0.1524" layer="91"/>
+<pinref part="R2" gate="G$1" pin="2"/>
+<pinref part="C5" gate="G$1" pin="1"/>
+<junction x="119.38" y="55.88"/>
+</segment>
+</net>
+<net name="N$7" class="0">
+<segment>
+<pinref part="C5" gate="G$1" pin="2"/>
+<wire x1="127" y1="55.88" x2="137.16" y2="55.88" width="0.1524" layer="91"/>
+<wire x1="137.16" y1="55.88" x2="137.16" y2="68.58" width="0.1524" layer="91"/>
+<wire x1="137.16" y1="68.58" x2="160.02" y2="68.58" width="0.1524" layer="91"/>
+<pinref part="U$2" gate="G$1" pin="IN+"/>
+<wire x1="160.02" y1="68.58" x2="160.02" y2="63.5" width="0.1524" layer="91"/>
+</segment>
+</net>
+<net name="N$8" class="0">
+<segment>
+<pinref part="C6" gate="G$1" pin="2"/>
+<wire x1="127" y1="45.72" x2="137.16" y2="45.72" width="0.1524" layer="91"/>
+<wire x1="137.16" y1="45.72" x2="137.16" y2="35.56" width="0.1524" layer="91"/>
+<wire x1="137.16" y1="35.56" x2="149.86" y2="35.56" width="0.1524" layer="91"/>
+<pinref part="U$2" gate="G$1" pin="IN-"/>
+<wire x1="149.86" y1="35.56" x2="149.86" y2="43.18" width="0.1524" layer="91"/>
+</segment>
+</net>
+<net name="N$9" class="0">
+<segment>
+<pinref part="U$2" gate="G$1" pin="VPS"/>
+<wire x1="154.94" y1="63.5" x2="154.94" y2="81.28" width="0.1524" layer="91"/>
+<wire x1="154.94" y1="81.28" x2="152.4" y2="81.28" width="0.1524" layer="91"/>
+<pinref part="U$2" gate="G$1" pin="ENB"/>
+<wire x1="152.4" y1="81.28" x2="147.32" y2="81.28" width="0.1524" layer="91"/>
+<wire x1="152.4" y1="63.5" x2="152.4" y2="81.28" width="0.1524" layer="91"/>
+<junction x="152.4" y="81.28"/>
+<pinref part="C7" gate="G$1" pin="2"/>
+<pinref part="L2" gate="G$1" pin="1"/>
+<junction x="147.32" y="81.28"/>
+</segment>
+</net>
+<net name="5V" class="0">
+<segment>
+<pinref part="L2" gate="G$1" pin="2"/>
+<wire x1="137.16" y1="81.28" x2="127" y2="81.28" width="0.1524" layer="91"/>
+<label x="127" y="83.82" size="1.778" layer="95"/>
+</segment>
+<segment>
+<pinref part="J3" gate="G$1" pin="4"/>
+<wire x1="99.06" y1="93.98" x2="104.14" y2="93.98" width="0.1524" layer="91"/>
+<label x="106.68" y="93.98" size="1.778" layer="95"/>
+</segment>
+<segment>
+<pinref part="L1" gate="G$1" pin="2"/>
+<wire x1="48.26" y1="81.28" x2="38.1" y2="81.28" width="0.1524" layer="91"/>
+<label x="38.1" y="83.82" size="1.778" layer="95"/>
+</segment>
+</net>
+<net name="OUT2" class="0">
+<segment>
+<pinref part="U$2" gate="G$1" pin="OUT"/>
+<wire x1="157.48" y1="43.18" x2="157.48" y2="35.56" width="0.1524" layer="91"/>
+<wire x1="157.48" y1="35.56" x2="170.18" y2="35.56" width="0.1524" layer="91"/>
+<pinref part="C8" gate="G$1" pin="2"/>
+<wire x1="170.18" y1="35.56" x2="177.8" y2="35.56" width="0.1524" layer="91"/>
+<junction x="170.18" y="35.56"/>
+<label x="177.8" y="38.1" size="1.778" layer="95"/>
+</segment>
+<segment>
+<pinref part="J3" gate="G$1" pin="1"/>
+<wire x1="99.06" y1="86.36" x2="104.14" y2="86.36" width="0.1524" layer="91"/>
+<label x="106.68" y="86.36" size="1.778" layer="95"/>
+</segment>
+</net>
